File: pcb/WaveGlideNG/_autosave-WaveGlideNG.kicad_pcb (KiCad board)
At the start: 2 copper layers, 107.1 x 71.6 mm, 22 parts

Commit message: footprints
Parts:
- STATUSRGB1: footprint LEDs:LED-L1T2_LUMILEDS -> WaveGlideNG:RGBA_5mm
- moved STATUSRGB1 13.1 mm to (279.2, 52.3), turned to 90 degrees
Connections:
- R3 pad 2: (no net) -> Net-(R3-Pad2)
Changed lines of the file:
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@@
     (zones 0)
     (modules 22)
-    (nets 28)
+    (nets 29)
   )
   (page A4)
@@
   (net 20 "Net-(R1-Pad2)")
   (net 21 "Net-(R2-Pad2)")
-  (net 22 "Net-(R4-Pad1)")
-  (net 23 PHOTO_CA)
-  (net 24 PHOTO_AN)
-  (net 25 RED_CA)
-  (net 26 RED_AN)
-  (net 27 POWERDISABLE)
+  (net 22 "Net-(R3-Pad2)")
+  (net 23 "Net-(R4-Pad1)")
+  (net 24 PHOTO_CA)
+  (net 25 PHOTO_AN)
+  (net 26 RED_CA)
+  (net 27 RED_AN)
+  (net 28 POWERDISABLE)
   (net_class Default "This is the default net class."
     (clearance 0.2)
@@
     (add_net "Net-(R1-Pad2)")
     (add_net "Net-(R2-Pad2)")
+    (add_net "Net-(R3-Pad2)")
     (add_net "Net-(R4-Pad1)")
     (add_net OUT_BLUE)
@@
     (pad 10 thru_hole oval (at 0 -22.86) (size 1.7 1.7) (drill 1) (layers *.Cu *.Mask))
     (pad 11 thru_hole oval (at 0 -25.4) (size 1.7 1.7) (drill 1) (layers *.Cu *.Mask)
-      (net 27 POWERDISABLE))
+      (net 28 POWERDISABLE))
     (pad 12 thru_hole oval (at 0 -27.94) (size 1.7 1.7) (drill 1) (layers *.Cu *.Mask)
       (net 8 /VBAT))
@@
     (fp_line (start -6.25 6.25) (end 6.25 6.25) (layer F.Fab) (width 0.1))
     (fp_line (start -6.25 -6.25) (end -6.25 6.25) (layer F.Fab) (width 0.1))
-    (pad 2 thru_hole oval (at 7.62 0) (size 2.4 2.4) (drill 1.2) (layers *.Cu *.Mask))
+    (pad 2 thru_hole oval (at 7.62 0) (size 2.4 2.4) (drill 1.2) (layers *.Cu *.Mask)
+      (net 22 "Net-(R3-Pad2)"))
     (pad 1 thru_hole circle (at 0 0) (size 2.4 2.4) (drill 1.2) (layers *.Cu *.Mask)
       (net 15 OUT_GREEN))
@@
     (fp_line (start 9.15 -6.6) (end -6.6 -6.6) (layer F.CrtYd) (width 0.05))
     (pad 1 thru_hole circle (at 0 0) (size 2.4 2.4) (drill 1.2) (layers *.Cu *.Mask)
-      (net 22 "Net-(R4-Pad1)"))
+      (net 23 "Net-(R4-Pad1)"))
     (pad 2 thru_hole oval (at 7.62 0) (size 2.4 2.4) (drill 1.2) (layers *.Cu *.Mask)
       (net 18 OUT_VALVE))
@@
       (at (xyz 0 0 0))
       (scale (xyz 0.393701 0.393701 0.393701))
-      (rotate (xyz 0 0 0))
-    )
-  )
-  (module LEDs:LED-L1T2_LUMILEDS (layer F.Cu)
-    (at 291.846 55.9054)
-    (descr http://www.lumileds.com/uploads/438/DS133-pdf)
-    (tags "LUMILEDS LUXEON TX L1T2 LED")
-    (attr smd)
-    (fp_text reference STATUSRGB1 (at 0 2.58) (layer F.SilkS)
-      (effects (font (size 1 1) (thickness 0.15)))
-    )
-    (fp_text value STATUSRGB (at 0 -3.42) (layer F.Fab)
-      (effects (font (size 1 1) (thickness 0.15)))
-    )
-    (fp_circle (center 0 -0.42) (end 0 -2.07) (layer F.Fab) (width 0.1))
-    (fp_line (start 1.4 1.5) (end -1.93 1.5) (layer F.SilkS) (width 0.12))
-    (fp_line (start 1.93 -2.35) (end 1.93 1.5) (layer F.SilkS) (width 0.12))
-    (fp_line (start -1.93 -2.35) (end 1.93 -2.35) (layer F.SilkS) (width 0.12))
-    (fp_line (start -1.93 1.5) (end -1.93 -2.35) (layer F.SilkS) (width 0.12))
-    (fp_line (start 2.25 1.83) (end -2.25 1.83) (layer F.CrtYd) (width 0.05))
-    (fp_line (start 2.25 -2.67) (end 2.25 1.83) (layer F.CrtYd) (width 0.05))
-    (fp_line (start -2.25 -2.67) (end 2.25 -2.67) (layer F.CrtYd) (width 0.05))
-    (fp_line (start -2.25 1.83) (end -2.25 -2.67) (layer F.CrtYd) (width 0.05))
-    (fp_line (start 1.8 1.4) (end 1.8 -2.2) (layer F.Fab) (width 0.1))
-    (fp_line (start -1.8 1.4) (end 1.8 1.4) (layer F.Fab) (width 0.1))
-    (fp_line (start -1.8 -2.2) (end -1.8 1.4) (layer F.Fab) (width 0.1))
-    (fp_line (start -1.8 -2.2) (end 1.8 -2.2) (layer F.Fab) (width 0.1))
-    (pad 3 smd rect (at 0 -0.52) (size 1.4 1.2) (layers F.Cu F.Paste F.Mask)
-      (net 21 "Net-(R2-Pad2)"))
-    (pad 2 smd rect (at -0.45 0.52) (size 0.55 0.38) (layers F.Cu F.Paste F.Mask)
-      (net 7 +3V3))
-    (pad 1 smd rect (at 0.45 0.52) (size 0.55 0.38) (layers F.Cu F.Paste F.Mask)
-      (net 20 "Net-(R1-Pad2)"))
-    (model ${KISYS3DMOD}/LEDs.3dshapes/LED-L1T2_LUMILEDS.wrl
-      (at (xyz 0 0 0))
-      (scale (xyz 1 1 1))
       (rotate (xyz 0 0 0))
     )
@@
       (net 6 GND))
     (pad 1 thru_hole rect (at 0 0) (size 1.7 1.7) (drill 1) (layers *.Cu *.Mask)
-      (net 22 "Net-(R4-Pad1)"))
+      (net 23 "Net-(R4-Pad1)"))
     (model ${KISYS3DMOD}/Pin_Headers.3dshapes/Pin_Header_Straight_1x02_Pitch2.54mm.wrl
       (at (xyz 0 0 0))
@@
     (fp_line (start -0.635 -1.27) (end 1.27 -1.27) (layer F.Fab) (width 0.1))
     (pad 5 thru_hole oval (at 0 10.16 90) (size 1.7 1.7) (drill 1) (layers *.Cu *.Mask)
-      (net 23 PHOTO_CA))
+      (net 24 PHOTO_CA))
     (pad 4 thru_hole oval (at 0 7.62 90) (size 1.7 1.7) (drill 1) (layers *.Cu *.Mask)
-      (net 24 PHOTO_AN))
+      (net 25 PHOTO_AN))
     (pad 3 thru_hole oval (at 0 5.08 90) (size 1.7 1.7) (drill 1) (layers *.Cu *.Mask)
       (net 6 GND))
     (pad 2 thru_hole oval (at 0 2.54 90) (size 1.7 1.7) (drill 1) (layers *.Cu *.Mask)
-      (net 25 RED_CA))
+      (net 26 RED_CA))
     (pad 1 thru_hole rect (at 0 0 90) (size 1.7 1.7) (drill 1) (layers *.Cu *.Mask)
-      (net 26 RED_AN))
+      (net 27 RED_AN))
     (model ${KISYS3DMOD}/Pin_Headers.3dshapes/Pin_Header_Straight_1x05_Pitch2.54mm.wrl
       (at (xyz 0 0 0))
@@
     (fp_line (start -7.112 -12.7) (end -6.096 -12.7) (layer Dwgs.User) (width 0.12))
     (pad 1 thru_hole circle (at -4.5 -2.5) (size 2.2 2.2) (drill 1.3) (layers *.Cu *.Mask)
-      (net 27 POWERDISABLE))
+      (net 28 POWERDISABLE))
     (pad 2 thru_hole circle (at -4.5 -5.7) (size 2.2 2.2) (drill 1.3) (layers *.Cu *.Mask)
       (net 6 GND))
@@
       (net 6 GND))
     (pad 2 thru_hole circle (at 2.77 0 180) (size 2 2) (drill 1.1) (layers *.Cu *.Mask)
-      (net 25 RED_CA))
+      (net 26 RED_CA))
     (pad 3 thru_hole circle (at 0 0 180) (size 2 2) (drill 1.1) (layers *.Cu *.Mask)
-      (net 26 RED_AN))
+      (net 27 RED_AN))
     (pad 4 thru_hole circle (at -2.77 0 180) (size 2 2) (drill 1.1) (layers *.Cu *.Mask)
       (net 12 IN_USER1))
     (pad 5 thru_hole circle (at -5.54 0 180) (size 2 2) (drill 1.1) (layers *.Cu *.Mask)
-      (net 24 PHOTO_AN))
+      (net 25 PHOTO_AN))
     (pad 6 thru_hole circle (at 4.15 2.84 180) (size 2 2) (drill 1.1) (layers *.Cu *.Mask)
       (net 6 GND))
@@
       (net 11 IN_USER2))
     (pad 9 thru_hole circle (at -4.15 2.84 180) (size 2 2) (drill 1.1) (layers *.Cu *.Mask)
-      (net 23 PHOTO_CA))
+      (net 24 PHOTO_CA))
     (pad 10 thru_hole circle (at 12.5 1.42 180) (size 4.8 4.8) (drill 3.2) (layers *.Cu *.Mask))
     (pad 11 thru_hole circle (at -12.5 1.42 180) (size 4.8 4.8) (drill 3.2) (layers *.Cu *.Mask))
   )
+  (module WaveGlideNG:RGBA_5mm (layer F.Cu)
+    (at 279.2476 52.2732 90)
+    (descr 604-WP154A43VBDZGWCA)
+    (fp_text reference STATUSRGB1 (at 0 5 90) (layer F.SilkS)
+      (effects (font (size 1 1) (thickness 0.15)))
+    )
+    (fp_text value STATUSRGB (at 0 -5 90) (layer F.Fab)
+      (effects (font (size 1 1) (thickness 0.15)))
+    )
+    (fp_circle (center 0 0) (end 3 0) (layer Dwgs.User) (width 0.12))
+    (fp_line (start -1.5 -2.6) (end 1.5 -2.6) (layer Dwgs.User) (width 0.12))
+    (pad 1 thru_hole oval (at 0 -1.905 90) (size 2 1) (drill 0.7) (layers *.Cu *.Mask)
+      (net 20 "Net-(R1-Pad2)"))
+    (pad 2 thru_hole oval (at 0 -0.625 90) (size 2 1) (drill 0.7) (layers *.Cu *.Mask)
+      (net 7 +3V3))
+    (pad 3 thru_hole oval (at 0 0.635 90) (size 2 1) (drill 0.7) (layers *.Cu *.Mask)
+      (net 21 "Net-(R2-Pad2)"))
+    (pad 4 thru_hole oval (at 0 1.905 90) (size 2 1) (drill 0.7) (layers *.Cu *.Mask)
+      (net 22 "Net-(R3-Pad2)"))
+  )
   (gr_circle (center 220.402401 90.706793) (end 220.002401 90.706793) (layer Dwgs.User) (width 0.2))
