File: pcb/WaveGlideNG/WaveGlideNG.kicad_pcb (KiCad board)
At the start: 2 copper layers, 107.1 x 71.6 mm, 22 parts

Commit message: footprints
Parts:
- added VALVECONN2: VALVECONN, WaveGlideNG:VALECONN, F.Cu at (146.0, 136.0)
- D1: footprint Diodes_ThroughHole:D_5KPW_P12.70mm_Horizontal -> Diodes_ThroughHole:D_A-405_P10.16mm_Horizontal
- R1, R2, R3, R4: footprint Resistors_ThroughHole:R_Axial_Power_L48.0mm_W12.5mm_P7.62mm_Vertical -> Resistors_ThroughHole:R_Axial_DIN0207_L6.3mm_D2.5mm_P10.16mm_Horizontal
- STATUSRGB1: footprint LEDs:LED-L1T2_LUMILEDS -> WaveGlideNG:RGBA_5mm
- VALVECONN1: footprint Pin_Headers:Pin_Header_Straight_1x02_Pitch2.54mm -> WaveGlideNG:VALECONN
- VALVESSR1: footprint Pin_Headers:Pin_Header_Straight_1x02_Pitch2.54mm -> WaveGlideNG:SSR
- moved R3 280.1 mm to (112.2, 118.6), turned to 90 degrees
- moved VALVESSR1 256.1 mm to (124.0, 133.6)
- moved R4 255.7 mm to (118.0, 139.0), turned to 90 degrees
- moved R2 250.8 mm to (98.0, 117.8)
- moved R1 227.0 mm to (98.0, 114.0)
- moved VALVECONN1 218.0 mm to (146.0, 111.0)
- moved YS2000PROBE1 197.7 mm to (104.8, 143.2)
- moved STATUSRGB1 181.7 mm to (112.0, 82.0), turned to 90 degrees
- moved BMP280 178.9 mm to (98.2, 123.0)
- moved BATCONN1 136.6 mm to (143.0, 107.0), turned to 90 degrees
- moved YS2000UART1 134.5 mm to (105.6, 91.2)
- moved D1 125.5 mm to (145.0, 117.0), turned to 270 degrees
- moved REF** 118.0 mm to (136.8, 123.9)
- moved REF** 118.0 mm to (119.0, 123.9)
- moved REF** 118.0 mm to (119.0, 78.1)
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Connections:
- R3 pad 2: (no net) -> Net-(R3-Pad2)
Other:
- board size 107.1 x 71.6 mm -> 72 x 70.6 mm

Commit message: footprints
Parts:
- moved DIFFPRESSURE1 1.34 mm to (102.6, 104.0)
- moved R2 1.20 mm to (98.0, 119.0)
- moved R1 1.00 mm to (98.0, 115.0)
- moved R3 0.40 mm to (112.2, 119.0)
Changed lines of the file:
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@@
     (pad 8 thru_hole circle (at 0 0) (size 2.4 2.4) (drill 1.4) (layers *.Cu *.Mask))
-  )
-  (module WaveGlideNG:DIFFPRESS (layer F.Cu)
-    (at 102 102.8 180)
-    (descr SSCMRRN001PDAA3)
-    (fp_text reference DIFFPRESSURE1 (at -6.11 0 90) (layer F.SilkS)
-      (effects (font (size 1 1) (thickness 0.15)))
-    )
-    (fp_text value PressSensor (at 0 0) (layer F.Fab)
-      (effects (font (size 1 1) (thickness 0.15)))
-    )
-    (fp_line (start -5.11 9.15) (end 5.109999 9.15) (layer F.SilkS) (width 0.12))
-    (fp_line (start 5.109999 9.15) (end 5.11 -9.15) (layer F.SilkS) (width 0.12))
-    (fp_line (start 5.11 -9.15) (end -5.109999 -9.15) (layer F.SilkS) (width 0.12))
-    (fp_line (start -5.109999 -9.15) (end -5.11 -3.05) (layer F.SilkS) (width 0.12))
-    (fp_line (start -5.11 -3.05) (end -4.75 -3.05) (layer F.SilkS) (width 0.12))
-    (fp_line (start -4.75 -3.05) (end -4.75 3.049999) (layer F.SilkS) (width 0.12))
-    (fp_line (start -4.75 3.049999) (end -5.11 3.049999) (layer F.SilkS) (width 0.12))
-    (fp_line (start -5.11 3.049999) (end -5.11 9.15) (layer F.SilkS) (width 0.12))
-    (fp_line (start -4.86 -8.9) (end 4.86 -8.9) (layer F.CrtYd) (width 0.05))
-    (fp_line (start 4.86 -8.9) (end 4.86 8.9) (layer F.CrtYd) (width 0.05))
-    (fp_line (start 4.86 8.9) (end -4.86 8.9) (layer F.CrtYd) (width 0.05))
-    (fp_line (start -4.86 8.9) (end -4.86 -8.9) (layer F.CrtYd) (width 0.05))
-    (pad 8 thru_hole oval (at -3.81 -6.65 180) (size 1.6 4) (drill 0.8) (layers *.Cu *.Mask))
-    (pad 1 thru_hole oval (at -3.81 6.65 180) (size 1.6 4) (drill 0.8) (layers *.Cu *.Mask))
-    (pad 7 thru_hole oval (at -1.27 -6.65 180) (size 1.6 4) (drill 0.8) (layers *.Cu *.Mask))
-    (pad 2 thru_hole oval (at -1.27 6.65 180) (size 1.6 4) (drill 0.8) (layers *.Cu *.Mask)
-      (net 7 +3V3))
-    (pad 6 thru_hole oval (at 1.27 -6.65 180) (size 1.6 4) (drill 0.8) (layers *.Cu *.Mask))
-    (pad 3 thru_hole oval (at 1.27 6.65 180) (size 1.6 4) (drill 0.8) (layers *.Cu *.Mask)
-      (net 10 IN_DIFFPRES))
-    (pad 5 thru_hole oval (at 3.81 -6.65 180) (size 1.6 4) (drill 0.8) (layers *.Cu *.Mask))
-    (pad 4 thru_hole oval (at 3.81 6.65 180) (size 1.6 4) (drill 0.8) (layers *.Cu *.Mask)
-      (net 6 GND))
   )
   (module WaveGlideNG:PIEZO (layer F.Cu)
@@
   )
   (module Resistors_ThroughHole:R_Axial_DIN0207_L6.3mm_D2.5mm_P10.16mm_Horizontal (layer F.Cu)
-    (at 98 114)
+    (at 98 115)
     (descr "Resistor, Axial_DIN0207 series, Axial, Horizontal, pin pitch=10.16mm, 0.25W = 1/4W, length*diameter=6.3*2.5mm^2, http://cdn-reichelt.de/documents/datenblatt/B400/1_4W%23YAG.pdf")
     (tags "Resistor Axial_DIN0207 series Axial Horizontal pin pitch 10.16mm 0.25W = 1/4W length 6.3mm diameter 2.5mm")
@@
   )
   (module Resistors_ThroughHole:R_Axial_DIN0207_L6.3mm_D2.5mm_P10.16mm_Horizontal (layer F.Cu)
-    (at 98 117.8)
+    (at 98 119)
     (descr "Resistor, Axial_DIN0207 series, Axial, Horizontal, pin pitch=10.16mm, 0.25W = 1/4W, length*diameter=6.3*2.5mm^2, http://cdn-reichelt.de/documents/datenblatt/B400/1_4W%23YAG.pdf")
     (tags "Resistor Axial_DIN0207 series Axial Horizontal pin pitch 10.16mm 0.25W = 1/4W length 6.3mm diameter 2.5mm")
@@
   )
   (module Resistors_ThroughHole:R_Axial_DIN0207_L6.3mm_D2.5mm_P10.16mm_Horizontal (layer F.Cu)
-    (at 112.2 118.6 90)
+    (at 112.2 119 90)
     (descr "Resistor, Axial_DIN0207 series, Axial, Horizontal, pin pitch=10.16mm, 0.25W = 1/4W, length*diameter=6.3*2.5mm^2, http://cdn-reichelt.de/documents/datenblatt/B400/1_4W%23YAG.pdf")
     (tags "Resistor Axial_DIN0207 series Axial Horizontal pin pitch 10.16mm 0.25W = 1/4W length 6.3mm diameter 2.5mm")
@@
       (net 6 GND))
   )
+  (module WaveGlideNG:DIFFPRESS (layer F.Cu)
+    (at 102.6 104 180)
+    (descr SSCMRRN001PDAA3)
+    (fp_text reference DIFFPRESSURE1 (at -6.11 0 90) (layer F.SilkS)
+      (effects (font (size 1 1) (thickness 0.15)))
+    )
+    (fp_text value PressSensor (at 0 0) (layer F.Fab)
+      (effects (font (size 1 1) (thickness 0.15)))
+    )
+    (fp_line (start -5.11 9.15) (end 5.109999 9.15) (layer F.SilkS) (width 0.12))
+    (fp_line (start 5.109999 9.15) (end 5.11 -9.15) (layer F.SilkS) (width 0.12))
+    (fp_line (start 5.11 -9.15) (end -5.109999 -9.15) (layer F.SilkS) (width 0.12))
+    (fp_line (start -5.109999 -9.15) (end -5.11 -3.05) (layer F.SilkS) (width 0.12))
+    (fp_line (start -5.11 -3.05) (end -4.75 -3.05) (layer F.SilkS) (width 0.12))
+    (fp_line (start -4.75 -3.05) (end -4.75 3.049999) (layer F.SilkS) (width 0.12))
+    (fp_line (start -4.75 3.049999) (end -5.11 3.049999) (layer F.SilkS) (width 0.12))
+    (fp_line (start -5.11 3.049999) (end -5.11 9.15) (layer F.SilkS) (width 0.12))
+    (fp_line (start -4.86 -8.9) (end 4.86 -8.9) (layer F.CrtYd) (width 0.05))
+    (fp_line (start 4.86 -8.9) (end 4.86 8.9) (layer F.CrtYd) (width 0.05))
+    (fp_line (start 4.86 8.9) (end -4.86 8.9) (layer F.CrtYd) (width 0.05))
+    (fp_line (start -4.86 8.9) (end -4.86 -8.9) (layer F.CrtYd) (width 0.05))
+    (pad 8 thru_hole oval (at -3.81 -6.65 180) (size 1.6 3) (drill 0.8) (layers *.Cu *.Mask))
+    (pad 1 thru_hole oval (at -3.81 6.65 180) (size 1.6 3) (drill 0.8) (layers *.Cu *.Mask))
+    (pad 7 thru_hole oval (at -1.27 -6.65 180) (size 1.6 3) (drill 0.8) (layers *.Cu *.Mask))
+    (pad 2 thru_hole oval (at -1.27 6.65 180) (size 1.6 3) (drill 0.8) (layers *.Cu *.Mask)
+      (net 7 +3V3))
+    (pad 6 thru_hole oval (at 1.27 -6.65 180) (size 1.6 3) (drill 0.8) (layers *.Cu *.Mask))
+    (pad 3 thru_hole oval (at 1.27 6.65 180) (size 1.6 3) (drill 0.8) (layers *.Cu *.Mask)
+      (net 10 IN_DIFFPRES))
+    (pad 5 thru_hole oval (at 3.81 -6.65 180) (size 1.6 3) (drill 0.8) (layers *.Cu *.Mask))
+    (pad 4 thru_hole oval (at 3.81 6.65 180) (size 1.6 3) (drill 0.8) (layers *.Cu *.Mask)
+      (net 6 GND))
+  )

Commit message: v0.1 PCB ordered
Parts:
- added BATCONN2: BAT-, WaveGlideNG:VALECONN, F.Cu at (140.0, 144.0)
- BATCONN1: value BATCONN -> BAT+; footprint Pin_Headers:Pin_Header_Straight_1x02_Pitch2.54mm -> WaveGlideNG:VALECONN
- POWERSWITCH1: value POWERSWITCH -> PWRSWITCH
- moved BATCONN1 37.7 mm to (136.0, 144.0)
- moved REF** 28.4 mm to (98.2, 143.2)
- moved REF** 25.0 mm to (143.7, 102.2)
- moved REF** 23.7 mm to (99.2, 91.2)
- moved BMP280 21.6 mm to (113.6, 138.2), turned to 180 degrees
- moved REF** 20.4 mm to (130.2, 143.2)
- moved YS2000PROBE1 10.2 mm to (115.0, 143.2), turned to 270 degrees
- moved D1 6.00 mm to (145.0, 123.0)
- moved VALVECONN1 6.00 mm to (146.0, 117.0)
- moved VALVECONN2 3.00 mm to (146.0, 139.0)
- moved R2 1.12 mm to (99.0, 118.5)
- moved R1 1.00 mm to (99.0, 115.0)
- moved STATUSRGB1 1.00 mm to (112.0, 83.0)
Routing:
- net +3V3: track 0.00 -> 86.7 mm
- net RED_AN: track 0.00 -> 78.4 mm
- net RED_CA: track 0.00 -> 70.7 mm
- net PHOTO_AN: track 0.00 -> 68.1 mm
- net PHOTO_CA: track 0.00 -> 65.0 mm
- net /VBAT: track 0.00 -> 63.8 mm
- net OUT_BLUE: track 0.00 -> 49.4 mm
- net OUT_RED: track 0.00 -> 48.6 mm
- net IN_USER2: track 0.00 -> 43.9 mm
- net Net-(R2-Pad2): track 0.00 -> 42.5 mm
- net OUT_BMP280_CS: track 0.00 -> 41.5 mm
- net /TX: track 0.00 -> 41.0 mm
- net OUT_VALVE: track 0.00 -> 40.2 mm
- net IN_USER1: track 0.00 -> 39.9 mm
- net /RX: track 0.00 -> 36.8 mm
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- added copper zone on B.Cu, net GND
Other:
- board size 72 x 70.6 mm -> 72 x 70 mm
- net class Default: clearance 0.2 -> 0.25
- net class Power: clearance 0.4 -> 0.5
- rule trace_clearance: 0.2 -> 0.25
- rule trace_min: 0.2 -> 0.25
- board text added: "(c) 2019 Nortd Labs"
- board text added: "WaveglideNG"
- board text added: "v0.1"
