File: pcb/WaveGlideNG/WaveGlideNG.sch (KiCad schematic (older format))
At the start: 22 parts, among them J1 feather long, J2 feather short

Commit message: footprints
Parts:
- removed PowerSwitch: SW_SPST, symbol Switch:SW_SPST
- added POWERSWITCH1: POWERSWITCH, WaveGlideNG:TE_Switch, symbol Connector_Generic:Conn_01x08
- BATCONN1: renamed from J?; value BatConn -> BATCONN; footprint (none) -> Pin_Headers:Pin_Header_Straight_1x02_Pitch2.54mm
- BMP280: renamed from J?; footprint (none) -> Pin_Headers:Pin_Header_Straight_1x07_Pitch2.54mm
- D1: renamed from D?; footprint (none) -> Diodes_ThroughHole:D_5KPW_P12.70mm_Horizontal
- DIFFPRESSURE1: renamed from J?; footprint (none) -> WaveGlideNG:DIFFPRESS
- FEATHERBLELONG1: renamed from J1; value feather long -> FEATHERBLELONG
- FEATHERBLESHORT1: renamed from J2; value feather short -> FEATHERBLESHORT
- PIEZOCONN1: renamed from J?; value PiezoSpeaker -> PIEZOCONN; footprint (none) -> WaveGlideNG:PIEZO
- PROBEJACK1: renamed from J?; value PulsOxyProbe -> PROBEJACK; footprint (none) -> WaveGlideNG:DB9HARTING
- R1, R2, R3: footprint (none) -> Resistors_ThroughHole:R_Axial_Power_L48.0mm_W12.5mm_P7.62mm_Vertical
- R4: renamed from R?; value R -> 360; footprint (none) -> Resistors_ThroughHole:R_Axial_Power_L48.0mm_W12.5mm_P7.62mm_Vertical
- STATUSRGB1: renamed from StatusRBG; value LED_RGBA -> STATUSRGB; footprint (none) -> WaveGlideNG:RGBA_5mm
- VALVECONN1: renamed from J?; value ValveConn -> VALVECONN; footprint (none) -> Pin_Headers:Pin_Header_Straight_1x02_Pitch2.54mm
- VALVESSR1: renamed from J?; value SSR -> VALVESSR; footprint (none) -> Pin_Headers:Pin_Header_Straight_1x02_Pitch2.54mm
- YS2000PROBE1: renamed from J?; value YS2000_B -> YS2000PROBE; footprint (none) -> Pin_Headers:Pin_Header_Straight_1x05_Pitch2.54mm
- YS2000UART1: renamed from J?; value YS2000_A -> YS2000UART; footprint (none) -> Pin_Headers:Pin_Header_Straight_1x04_Pitch2.54mm
Connections:
- net A1 is gone; now on net IN_USER1: FEATHERBLELONG1.11 (Pin_11)
- net A2 is gone; now on net IN_USER2: FEATHERBLELONG1.10 (Pin_10)
- net A4 is gone; now on net IN_DIFFPRES: FEATHERBLELONG1.8 (Pin_8)
- net BMP280_CS is gone; now on net OUT_BMP280_CS: FEATHERBLELONG1.7 (Pin_7)
- net P10 is gone; now on net OUT_GREEN: FEATHERBLESHORT1.6 (Pin_6)
- net P11 is gone; now on net OUT_BLUE: FEATHERBLESHORT1.7 (Pin_7)
- net P12 is gone; now on net OUT_RED: FEATHERBLESHORT1.8 (Pin_8)
- net P13 is gone; now on net OUT_VALVE: FEATHERBLESHORT1.9 (Pin_9)
- net P5 is gone; now on net OUT_PIEZO1: FEATHERBLESHORT1.3 (Pin_3)
- net P6 is gone; now on net OUT_PIEZO2: FEATHERBLESHORT1.4 (Pin_4)
- net GND: now also POWERSWITCH1.2 (Pin_2)
- net OUT_BLUE: now also R2.1; no longer R2.2
- net OUT_GREEN: now also R3.1; no longer R3.2
- net OUT_RED: now also R1.1; no longer R1.2
- net VBAT: now also BATCONN1.1 (Pin_1)
- net at STATUSRGB1.1 (RK): now also R1.2; no longer R1.1
- net at STATUSRGB1.3 (BK): now also R2.2; no longer R2.1
- net at STATUSRGB1.4 (GB): now also R3.2; no longer R3.1
- net EN renamed POWERDISABLE
- net POWERDISABLE: now also POWERSWITCH1.1 (Pin_1)
- no-connect marks 7 -> 22
Other:
- moved on the sheet: BATCONN1, BMP280, D1, DIFFPRESSURE1, H1, H2, H3, H4, PIEZOCONN1, PROBEJACK1, R1, R2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

Commit message: footprints
Parts:
- removed VALVECONN1: VALVECONN, Pin_Headers:Pin_Header_Straight_1x02_Pitch2.54mm, symbol Connector_Generic:Conn_01x02
- added VALVECONN1, VALVECONN2: VALVECONN, WaveGlideNG:VALECONN, symbol Connector_Generic:Conn_01x01
- D1: footprint Diodes_ThroughHole:D_5KPW_P12.70mm_Horizontal -> Diodes_ThroughHole:D_A-405_P10.16mm_Horizontal
- R1, R2, R3, R4: footprint Resistors_ThroughHole:R_Axial_Power_L48.0mm_W12.5mm_P7.62mm_Vertical -> Resistors_ThroughHole:R_Axial_DIN0207_L6.3mm_D2.5mm_P10.16mm_Horizontal
- VALVESSR1: footprint Pin_Headers:Pin_Header_Straight_1x02_Pitch2.54mm -> WaveGlideNG:SSR
Connections:
- net GND: now also VALVECONN2.1 (Pin_1)
- net at D1.1 (K), VALVESSR1.3 (Pin_3): now also VALVECONN1.1 (Pin_1)
Changed lines of the file:
@@
 F 0 "D1" H 9350 3376 50  0000 C CNN
 F 1 "D" H 9350 3375 50  0001 C CNN
-F 2 "Diodes_ThroughHole:D_5KPW_P12.70mm_Horizontal" H 9350 3500 50  0001 C CNN
+F 2 "Diodes_ThroughHole:D_A-405_P10.16mm_Horizontal" H 9350 3500 50  0001 C CNN
 F 3 "~" H 9350 3500 50  0001 C CNN
 	1    9350 3500
@@
 F 0 "R4" V 8450 3050 50  0000 C CNN
 F 1 "360" V 8550 3050 50  0000 C CNN
-F 2 "Resistors_ThroughHole:R_Axial_Power_L48.0mm_W12.5mm_P7.62mm_Vertical" V 8480 3050 50  0001 C CNN
+F 2 "Resistors_ThroughHole:R_Axial_DIN0207_L6.3mm_D2.5mm_P10.16mm_Horizontal" V 8480 3050 50  0001 C CNN
 F 3 "~" H 8550 3050 50  0001 C CNN
 	1    8550 3050
-	0    1    1    0
-$EndComp
-$Comp
-L Connector_Generic:Conn_01x02 VALVECONN1
-U 1 1 5D7CE25E
-P 9300 3950
-F 0 "VALVECONN1" V 9300 4050 50  0000 L CNN
-F 1 "VALVECONN" V 9263 4030 50  0001 L CNN
-F 2 "Pin_Headers:Pin_Header_Straight_1x02_Pitch2.54mm" H 9300 3950 50  0001 C CNN
-F 3 "~" H 9300 3950 50  0001 C CNN
-	1    9300 3950
 	0    1    1    0
 $EndComp
@@
 F 0 "VALVESSR1" H 9250 3250 50  0000 C CNN
 F 1 "VALVESSR" H 9250 3176 50  0001 C CNN
-F 2 "Pin_Headers:Pin_Header_Straight_1x02_Pitch2.54mm" H 9200 3050 50  0001 C CNN
+F 2 "WaveGlideNG:SSR" H 9200 3050 50  0001 C CNN
 F 3 "~" H 9200 3050 50  0001 C CNN
 	1    9200 3050
@@
 	9650 3050 9500 3050
 Wire Wire Line
-	9200 3750 9200 3500
-Wire Wire Line
-	9200 3500 8700 3500
-Connection ~ 9200 3500
+	9200 3500 9150 3500
 Connection ~ 8700 3500
 Wire Wire Line
@@
 F 0 "R1" H 4150 1500 50  0000 R CNN
 F 1 "120" H 4200 1600 50  0000 R CNN
-F 2 "Resistors_ThroughHole:R_Axial_Power_L48.0mm_W12.5mm_P7.62mm_Vertical" V 4030 1550 50  0001 C CNN
+F 2 "Resistors_ThroughHole:R_Axial_DIN0207_L6.3mm_D2.5mm_P10.16mm_Horizontal" V 4030 1550 50  0001 C CNN
 F 3 "~" H 4100 1550 50  0001 C CNN
 	1    4100 1550
@@
 F 0 "R2" H 4350 1500 50  0000 R CNN
 F 1 "30" H 4350 1600 50  0000 R CNN
-F 2 "Resistors_ThroughHole:R_Axial_Power_L48.0mm_W12.5mm_P7.62mm_Vertical" V 4230 1550 50  0001 C CNN
+F 2 "Resistors_ThroughHole:R_Axial_DIN0207_L6.3mm_D2.5mm_P10.16mm_Horizontal" V 4230 1550 50  0001 C CNN
 F 3 "~" H 4300 1550 50  0001 C CNN
 	1    4300 1550
@@
 F 0 "R3" H 4550 1500 50  0000 R CNN
 F 1 "10" H 4550 1600 50  0000 R CNN
-F 2 "Resistors_ThroughHole:R_Axial_Power_L48.0mm_W12.5mm_P7.62mm_Vertical" V 4430 1550 50  0001 C CNN
+F 2 "Resistors_ThroughHole:R_Axial_DIN0207_L6.3mm_D2.5mm_P10.16mm_Horizontal" V 4430 1550 50  0001 C CNN
 F 3 "~" H 4500 1550 50  0001 C CNN
 	1    4500 1550
@@
 Wire Wire Line
 	7600 1150 7750 1150
+$Comp
+L Connector_Generic:Conn_01x01 VALVECONN2
+U 1 1 5DD55E98
+P 9150 4050
+F 0 "VALVECONN2" V 9250 3650 50  0000 L CNN
+F 1 "VALVECONN" V 9350 3700 50  0001 L CNN
+F 2 "WaveGlideNG:VALECONN" H 9150 4050 50  0001 C CNN
+F 3 "~" H 9150 4050 50  0001 C CNN
+	1    9150 4050
+	0    1    1    0
+$EndComp
+$Comp
+L Connector_Generic:Conn_01x01 VALVECONN1
+U 1 1 5DD55101
+P 9300 4050
+F 0 "VALVECONN1" V 9400 4000 50  0000 L CNN
+F 1 "VALVECONN" H 9380 4001 50  0001 L CNN
+F 2 "WaveGlideNG:VALECONN" H 9300 4050 50  0001 C CNN
+F 3 "~" H 9300 4050 50  0001 C CNN
+	1    9300 4050
+	0    1    1    0
+$EndComp
+Wire Wire Line
+	9150 3850 9150 3500
+Connection ~ 9150 3500
+Wire Wire Line
+	9150 3500 8700 3500
+Wire Wire Line
+	9300 3850 9300 3750
 $EndSCHEMATC

Commit message: v0.1 PCB ordered
Parts:
- removed BATCONN1: BATCONN, Pin_Headers:Pin_Header_Straight_1x02_Pitch2.54mm, symbol Connector_Generic:Conn_01x02
- added BATCONN1: BAT+, WaveGlideNG:VALECONN, symbol Connector_Generic:Conn_01x01
- added BATCONN2: BAT-, WaveGlideNG:VALECONN, symbol Connector_Generic:Conn_01x01
Connections:
- net GND: now also BATCONN2.1 (Pin_1)
- net VBAT: now also BATCONN1.1 (Pin_1)
Changed lines of the file:
@@
-$EndComp
-$Comp
-L Connector_Generic:Conn_01x02 BATCONN1
-U 1 1 5D7CE8BD
-P 7500 4600
-F 0 "BATCONN1" H 7580 4546 50  0000 L CNN
-F 1 "BATCONN" H 7580 4501 50  0001 L CNN
-F 2 "Pin_Headers:Pin_Header_Straight_1x02_Pitch2.54mm" H 7500 4600 50  0001 C CNN
-F 3 "~" H 7500 4600 50  0001 C CNN
-	1    7500 4600
-	1    0    0    -1
 $EndComp
 $Comp
@@
 	3550 4200 3300 4200
 NoConn ~ 3550 4000
-Text Label 7050 4600 0    50   ~ 0
+Text Label 7050 4550 0    50   ~ 0
 VBAT
 $Comp
@@
 NoConn ~ 6550 2700
 Wire Wire Line
-	7050 4600 7300 4600
+	7050 4550 7300 4550
 NoConn ~ 1900 2000
 $Comp
@@
 Wire Wire Line
 	9300 3850 9300 3750
+$Comp
+L Connector_Generic:Conn_01x01 BATCONN1
+U 1 1 5DD86757
+P 7500 4550
+F 0 "BATCONN1" H 7600 4550 50  0001 L CNN
+F 1 "BAT+" H 7600 4550 50  0000 L CNN
+F 2 "WaveGlideNG:VALECONN" H 7500 4550 50  0001 C CNN
+F 3 "~" H 7500 4550 50  0001 C CNN
+	1    7500 4550
+	1    0    0    -1
+$EndComp
+$Comp
+L Connector_Generic:Conn_01x01 BATCONN2
+U 1 1 5DD872BD
+P 7500 4700
+F 0 "BATCONN2" H 7600 4700 50  0001 L CNN
+F 1 "BAT-" H 7600 4700 50  0000 L CNN
+F 2 "WaveGlideNG:VALECONN" H 7500 4700 50  0001 C CNN
+F 3 "~" H 7500 4700 50  0001 C CNN
+	1    7500 4700
+	1    0    0    -1
+$EndComp
 $EndSCHEMATC
