File: pcb/WaveGlide3X/WaveGlide3X.kicad_pcb (KiCad board)
At the start: 2 copper layers, 118 x 92 mm, 36 parts

Commit message: first pcb layout
Parts:
- removed BATCONN3: BAT+, WaveGlide3X:VALECONN
- removed BATCONN4: BAT-, WaveGlide3X:VALECONN
- removed FEATHERBLELONG1: FEATHERBLELONG, Pin_Headers:Pin_Header_Straight_1x16_Pitch2.54mm
- removed FEATHERBLESHORT1: FEATHERBLESHORT, Pin_Headers:Pin_Header_Straight_1x12_Pitch2.54mm
- removed H4: MountingHole, Mounting_Holes:MountingHole_4.3mm_M4_Pad_Via
- removed H5, H6: ValveMount M3, WaveGlide3X:VALECONN
- removed VALVECONN1, VALVECONN2: VALVECONN, WaveGlide3X:VALECONN
- removed YS2000UART1: YS2000UART, Pin_Headers:Pin_Header_Straight_1x04_Pitch2.54mm
- added AIRTEC1: AIRTEC, WaveGlide3X:Airtec_M20, F.Cu at (129.0, 139.0)
- BATCONN1: value BAT+ -> BATCONN; footprint WaveGlide3X:VALECONN -> WaveGlide3X:BATCONN
- BATCONN2: value BAT- -> BATCONN; footprint WaveGlide3X:VALECONN -> WaveGlide3X:BATCONN
- BMP280: footprint Pin_Headers:Pin_Header_Straight_1x07_Pitch2.54mm -> WaveGlide3X:Adafruit_BMP280
- CHARGER1: footprint Pin_Headers:Pin_Header_Straight_1x05_Pitch2.54mm -> WaveGlide3X:Adafruit_Charger_4410
- H1, H2, H3: footprint Mounting_Holes:MountingHole_4.3mm_M4_Pad_Via -> Mounting_Holes:MountingHole_3.2mm_M3_Pad_Via
- YS2000PROBE1: footprint Pin_Headers:Pin_Header_Straight_1x05_Pitch2.54mm -> WaveGlide3X:YS2000
- moved BATCONN1 177.4 mm to (99.0, 152.0)
- moved C2 171.0 mm to (72.0, 136.0)
- moved C1 157.0 mm to (72.0, 120.0)
- moved BATCONN2 149.1 mm to (119.0, 93.5), turned to 90 degrees
- moved H3 146.9 mm to (55.0, 113.0)
- moved R7 123.5 mm to (95.0, 146.0)
- moved VALVESSR1 123.5 mm to (82.0, 135.0), turned to 180 degrees
- moved D1 119.1 mm to (103.0, 141.0)
- moved YS2000PROBE1 116.2 mm to (49.0, 110.0)
- moved R1 115.6 mm to (64.0, 83.0), turned to 90 degrees
- moved H1 103.1 mm to (68.0, 66.0)
- moved R4 99.2 mm to (60.0, 104.0), turned to 90 degrees
- moved R2 99.0 mm to (69.0, 83.0), turned to 90 degrees
- moved BOOSTCONV1 93.1 mm to (72.0, 143.0), turned to 0 degrees
- moved R3 92.6 mm to (86.0, 86.0), turned to 180 degrees
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Connections:
- BATCONN2 pad 1: GND -> VBAT
- YS2000PROBE1 pad 1: RED_AN -> RX
- YS2000PROBE1 pad 2: RED_CA -> TX
- YS2000PROBE1 pad 3: GND -> +3V3
- YS2000PROBE1 pad 4: PHOTO_AN -> GND
- YS2000PROBE1 pad 5: PHOTO_CA -> RED_AN
Other:
- board size 118 x 92 mm -> 92 x 95 mm

Commit message: second pcb layout
Parts:
- AIRTEC1: footprint WaveGlide3X:Airtec_M20 -> WaveGlide3X:Airtec_M20_B
- moved BATCONN2 76.6 mm to (69.5, 152.0), turned to 0 degrees
- moved BMP280 53.9 mm to (85.0, 95.0)
- moved C2 45.6 mm to (116.0, 148.0), turned to 270 degrees
- moved DIFFPRESSURE1 45.2 mm to (81.0, 89.0), turned to 90 degrees
- moved PIEZOCONN1 42.1 mm to (110.5, 107.0)
- moved H3 39.2 mm to (79.0, 144.0)
- moved D1 30.5 mm to (83.0, 118.0), turned to 90 degrees
- moved R3 25.2 mm to (61.0, 83.0), turned to 90 degrees
- moved Feather_M0_BLE1 21.6 mm to (50.0, 96.0), turned to 270 degrees
- moved R7 20.1 mm to (113.0, 137.0), turned to 180 degrees
- moved BATCONN1 17.5 mm to (81.5, 152.0)
- moved BOOSTCONV1 17.0 mm to (89.0, 143.0)
- moved C1 16.6 mm to (81.0, 134.0), turned to 180 degrees
- moved R4 14.2 mm to (69.0, 93.0), turned to 180 degrees
- moved VALVESSR1 7.62 mm to (89.0, 138.0), turned to 270 degrees
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Other:
- board size 92 x 95 mm -> 89 x 95 mm
- board text added: "Waveglide3X v3.1"
- board text removed: "Waveglide3X"
- board text removed: "v0.1"

Commit message: before routing
Parts:
- DIFFPRESSURE1: value PressSensor -> DIFFPRESSURE
- moved D1 0.50 mm to (82.5, 118.0)
Other:
- board text added: "Waveglide3X"

Commit message: first routing
Parts:
- moved R4 35.4 mm to (86.0, 124.0)
- moved R1 4.00 mm to (69.0, 83.0)
- moved R2 4.00 mm to (65.0, 83.0)
Routing:
- net +3V3: track 0.00 -> 101.7 mm
- net VUSB: track 0.00 -> 97.4 mm
- net VUSB_SENSE: track 0.00 -> 89.7 mm
- net RX: track 0.00 -> 83.4 mm
- net TX: track 0.00 -> 77.3 mm
- net GND: track 0.00 -> 64.2 mm
- net OUT_PIEZO2: track 0.00 -> 53.8 mm
- net VBAT_ON: track 0.00 -> 53.7 mm
- net IN_USER2: track 0.00 -> 53.3 mm
- net IN_DIFFPRES: track 0.00 -> 50.9 mm
- net OUT_GREEN: track 0.00 -> 49.1 mm
- net OUT_PIEZO1: track 0.00 -> 48.3 mm
- net MOSI: track 0.00 -> 48.1 mm
- net IN_USER1: track 0.00 -> 48.1 mm
- net Net-(AIRTEC1-Pad1): track 0.00 -> 48.0 mm
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- added copper zone on B.Cu, net GND
- added copper zone on F.Cu, net VBAT

Commit message: roughly routed
Parts:
- DIFFPRESSURE1: value DIFFPRESSURE -> PressSensor
- moved R4 10.8 mm to (76.0, 128.0), turned to 90 degrees
- moved D1 10.0 mm to (83.0, 128.0)
Routing:
- net GND: track 64.2 -> 17.2 mm
- net TX: track 77.3 -> 91.6 mm
- net IN_USER2: track 53.3 -> 62.4 mm
- net VUSB: track 97.4 -> 89.5 mm, vias 0 -> 1
- net Net-(AIRTEC1-Pad1): track 48.0 -> 41.3 mm
- net OUT_PIEZO2: track 53.8 -> 59.8 mm
- net OUT_PIEZO1: track 48.3 -> 53.4 mm
- net VBAT_ON: track 53.7 -> 58.2 mm
- net OUT_RED: track 41.7 -> 45.7 mm
- net VUSB_SENSE: track 89.7 -> 92.9 mm, vias 0 -> 1
- net OUT_BLUE: track 44.9 -> 47.4 mm
- net IN_USER1: track 48.1 -> 49.6 mm
- net RX: track 83.4 -> 82.1 mm
- net MOSI: track 48.1 -> 47.2 mm

Commit message: configurable valve voltage added
Parts:
- added R8: 360, Resistors_ThroughHole:R_Axial_DIN0207_L6.3mm_D2.5mm_P10.16mm_Horizontal, F.Cu at (80.0, 128.0)
- added VALVESSR2: VALVESSR, WaveGlide3X:SSR, F.Cu at (116.5, 140.5)
- moved R7 1.58 mm to (112.5, 138.5)
- moved D1 1.50 mm to (84.5, 128.0)
- moved C2 0.50 mm to (116.0, 148.5)
Connections:
- Feather_M0_BLE1 pad 8: (no net) -> OUT_VCONV
- R7 pad 1: Net-(BOOSTCONV1-Pad3) -> Net-(R7-Pad1)
Routing:
- net Net-(R8-Pad1): track 0.00 -> 45.9 mm
- net OUT_VCONV: track 0.00 -> 39.1 mm
- net GND: track 17.2 -> 38.1 mm
- net Net-(R7-Pad1): track 0.00 -> 4.69 mm
- net +3V3: track 101.7 -> 105.3 mm
- net OUT_BMP280_CS: track 47.3 -> 50.6 mm
- net Net-(BOOSTCONV1-Pad3): track 17.6 -> 20.2 mm
- net IN_USER2: track 62.4 -> 60.6 mm
- net Net-(AIRTEC1-Pad1): track 41.3 -> 42.9 mm
- net OUT_PIEZO2: track 59.8 -> 61.4 mm
- net OUT_PIEZO1: track 53.4 -> 54.6 mm
- net VBAT_ON: track 58.2 -> 59.1 mm
Other:
- net class Power2 added: clearance 0.5, trace_width 1, via_dia 0.8, via_drill 0.4

Commit message: as exported
Parts:
- AIRTEC1: footprint WaveGlide3X:Airtec_M20_B -> WaveGlide3X:Airtec_M20_B_1MH
Routing:
- net GND: track 38.1 -> 40.3 mm
- net Net-(AIRTEC1-Pad1): track 42.9 -> 44.2 mm
Other:
- outline, holes or cut-outs redrawn
