File: pcb/WaveGlide3X/WaveGlide3X.kicad_pcb (KiCad board)
At the start: 2 copper layers, 89 x 95 mm, 29 parts

Commit message: changed feather footprint 180, routing
Parts:
- moved Feather_M0_BLE1 55.9 mm to (137.0, 135.0), turned to 90 degrees
- moved BATCONN2 2.42 mm to (136.0, 140.0)
- moved BATCONN1 0.50 mm to (146.0, 140.0)
Connections:
- Feather_M0_BLE1 pad 12: MISO -> MOSI
- Feather_M0_BLE1 pad 13: MOSI -> MISO
- YS2000PROBE1 pad 3: +3V3 -> GND
- YS2000PROBE1 pad 4: GND -> +3V3
Routing:
- net RX: track 82.6 -> 0.00 mm
- net IN_DIFFPRES: track 50.9 -> 0.00 mm
- net OUT_BMP280_CS: track 50.6 -> 0.00 mm
- net SCK: track 46.2 -> 0.00 mm
- net +3V3: track 105.3 -> 65.5 mm
- net MOSI: track 47.2 -> 17.4 mm
- net MISO: track 46.5 -> 17.4 mm
- net VBAT_ON: track 59.1 -> 88.2 mm
- net OUT_VCONV: track 39.1 -> 11.1 mm
- net TX: track 92.1 -> 70.2 mm
- net GND: track 40.3 -> 18.5 mm
- net VUSB: track 89.5 -> 71.0 mm, vias 1 -> 0
- net OUT_GREEN: track 49.1 -> 34.2 mm
- net OUT_BLUE: track 47.4 -> 33.9 mm
- net OUT_RED: track 45.7 -> 33.6 mm
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
Commit message: routing
Parts:
- added PIEZOCONN17: PIEZOCONN, WaveGlide3X:PIEZO_17, F.Cu at (177.0, 89.0)
- added Q1: KSC1815, Package_TO_SOT_THT:TO-92L_Inline_Wide, F.Cu at (174.0, 100.0)
- added R10: 1K, Resistor_THT:R_Axial_DIN0207_L6.3mm_D2.5mm_P10.16mm_Horizontal, F.Cu at (157.5, 81.0)
- added R9: 1K, Resistor_THT:R_Axial_DIN0207_L6.3mm_D2.5mm_P10.16mm_Horizontal, F.Cu at (182.0, 74.0)
- moved R6 3.50 mm to (178.5, 74.0)
- moved R5 1.00 mm to (175.0, 74.0)
Routing:
- net OUT_PIEZO2: track 57.0 -> 0.00 mm
- net IN_USER2: track 54.8 -> 7.22 mm
- net RX: track 0.00 -> 43.0 mm
- net VUSB: track 71.0 -> 102.9 mm
- net IN_USER1: track 45.3 -> 13.4 mm
- net Net-(PIEZOCONN17-Pad2): track 0.00 -> 29.9 mm
- net OUT_VALVE: track 3.24 -> 26.7 mm
- net OUT_PIEZO1: track 45.5 -> 68.4 mm
- net +3V3: track 65.5 -> 88.4 mm
- net Net-(Q1-Pad3): track 0.00 -> 21.9 mm
- net OUT_RED: track 33.6 -> 48.6 mm
- net OUT_BLUE: track 33.9 -> 45.4 mm
- net OUT_GREEN: track 34.2 -> 41.2 mm
- net GND: track 18.5 -> 14.6 mm
- net VUSB_SENSE: track 84.3 -> 81.9 mm
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Other:
- board text added: "(c) 2020 Nortd Labs"
- board text added: "Waveglide3X v3.2"
- board text removed: "(c) 2019 Nortd Labs"
- board text removed: "Waveglide3X v3.1"

Commit message: routing final touches
Routing:
- net IN_USER2: track 7.22 -> 79.4 mm, vias 0 -> 2
- net OUT_PIEZO2: track 0.00 -> 68.3 mm
- net +3V3: track 88.4 -> 152.6 mm, vias 0 -> 1
- net IN_USER1: track 13.4 -> 77.6 mm, vias 0 -> 2
- net IN_DIFFPRES: track 0.00 -> 53.7 mm
- net TX: track 70.2 -> 38.8 mm, vias 0 -> 1
- net SCK: track 0.00 -> 25.6 mm
- net OUT_BMP280_CS: track 0.00 -> 18.4 mm
- net VBAT_ON: track 88.2 -> 91.9 mm, vias 0 -> 1
- net VUSB_SENSE: track 81.9 -> 78.3 mm, vias 0 -> 1
- net RED_AN: track 39.8 -> 37.1 mm
- net OUT_BLUE: track 45.4 -> 44.6 mm
- net OUT_RED: track 48.6 -> 47.8 mm
- net VUSB: track 102.9 -> 102.2 mm
- net RX: track 43.0 -> 43.5 mm, vias 0 -> 1

Commit message: v3.2 as quoted
Parts:
- removed BATCONN2: BATCONN, WaveGlide3X:BATCONN
- moved BATCONN1 3.04 mm to (143.0, 140.0)
- moved Feather_M0_BLE1 0.28 mm to (136.9, 134.7)
Routing:
- net GND: track 14.6 -> 0.00 mm
- net IN_DIFFPRES: track 53.7 -> 44.7 mm
- net VUSB_SENSE: track 78.3 -> 82.6 mm
- net RX: track 43.5 -> 40.1 mm
- net OUT_PIEZO1: track 68.4 -> 71.7 mm
- net VBAT_ON: track 91.9 -> 88.9 mm
- net +3V3: track 152.6 -> 150.0 mm
- net SCK: track 25.6 -> 27.5 mm
- net IN_USER2: track 79.4 -> 80.9 mm
- net TX: track 38.8 -> 37.3 mm
- net OUT_GREEN: track 41.5 -> 43.0 mm
- net IN_USER1: track 77.6 -> 78.7 mm
- net Net-(Q1-Pad3): track 21.9 -> 22.7 mm
- net RED_AN: track 37.1 -> 36.4 mm
- net OUT_VCONV: track 11.1 -> 10.4 mm
Other:
- outline, holes or cut-outs redrawn
