File: pcb/WaveGlide3X/WaveGlide3X.sch (KiCad schematic (older format))
At the start: 34 parts

Commit message: first pcb layout
Parts:
- removed BATCONN1, BATCONN3: BAT+, WaveGlide3X:VALECONN, symbol Connector_Generic:Conn_01x01
- removed BATCONN2, BATCONN4: BAT-, WaveGlide3X:VALECONN, symbol Connector_Generic:Conn_01x01
- removed H4: MountingHole, Mounting_Holes:MountingHole_4.3mm_M4_Pad_Via, symbol Mechanical:MountingHole
- removed H5, H6: ValveMount M3, WaveGlide3X:VALECONN, symbol Mechanical:MountingHole
- removed VALVECONN1, VALVECONN2: VALVECONN, WaveGlide3X:VALECONN, symbol Connector_Generic:Conn_01x01
- removed YS2000PROBE1: YS2000PROBE, Pin_Headers:Pin_Header_Straight_1x05_Pitch2.54mm, symbol Connector_Generic:Conn_01x05
- removed YS2000UART1: YS2000UART, Pin_Headers:Pin_Header_Straight_1x04_Pitch2.54mm, symbol Connector_Generic:Conn_01x04
- added AIRTEC1: AIRTEC, WaveGlide3X:Airtec_M20, symbol Connector_Generic:Conn_01x02
- added BATCONN1, BATCONN2: BATCONN, WaveGlide3X:BATCONN, symbol Connector_Generic:Conn_01x02
- added YS2000PROBE1: YS2000PROBE, WaveGlide3X:YS2000, symbol Connector_Generic:Conn_01x09
- BMP280: footprint Pin_Headers:Pin_Header_Straight_1x07_Pitch2.54mm -> WaveGlide3X:Adafruit_BMP280
- CHARGER1: footprint Pin_Headers:Pin_Header_Straight_1x05_Pitch2.54mm -> WaveGlide3X:Adafruit_Charger_4410
- H1, H2, H3: footprint Mounting_Holes:MountingHole_4.3mm_M4_Pad_Via -> Mounting_Holes:MountingHole_3.2mm_M3_Pad_Via
Connections:
- net +3V3: now also YS2000PROBE1.3 (Pin_3)
- net GND: now also AIRTEC1.2 (Pin_2), BATCONN1.2 (Pin_2), BATCONN2.2 (Pin_2), YS2000PROBE1.4 (Pin_4), YS2000PROBE1.7 (Pin_7)
- net PHOTO_AN: now also YS2000PROBE1.8 (Pin_8)
- net PHOTO_CA: now also YS2000PROBE1.9 (Pin_9)
- net RED_AN: now also YS2000PROBE1.5 (Pin_5)
- net RED_CA: now also YS2000PROBE1.6 (Pin_6)
- net RX: now also YS2000PROBE1.1 (Pin_1)
- net TX: now also YS2000PROBE1.2 (Pin_2)
- net VBAT: now also BATCONN1.1 (Pin_1), BATCONN2.1 (Pin_1)
- net at BOOSTCONV1.4 (Pin_4), C2.1, D1.1 (K): now also AIRTEC1.1 (Pin_1)

Commit message: configurable valve voltage added
Parts:
- added R8: 360, Resistors_ThroughHole:R_Axial_DIN0207_L6.3mm_D2.5mm_P10.16mm_Horizontal, symbol Device:R
- added VALVESSR2: VALVESSR, WaveGlide3X:SSR, symbol Connector_Generic:Conn_02x02_Counter_Clockwise
- AIRTEC1: footprint WaveGlide3X:Airtec_M20 -> WaveGlide3X:Airtec_M20_B
Connections:
- net GND: now also VALVESSR2.2 (Pin_2)
- net at BOOSTCONV1.3 (Pin_3): now also VALVESSR2.3 (Pin_3); no longer R7.1
- net OUT_VCONV: now reaches Feather_M0_BLE1.8 (Pin_8)
- net OUT_VCONV: now also R8.2
- new net: R7.1, VALVESSR2.4 (Pin_4)
- new net: R8.1, VALVESSR2.1 (Pin_1)
- no-connect marks 19 -> 18
Changed lines of the file:
@@
 	8900 3800 8900 3950
-Wire Wire Line
-	9350 3950 9650 3950
-Wire Wire Line
-	9650 3950 9650 3800
 Wire Wire Line
 	9350 4350 9550 4350
@@
 Text GLabel 4850 2950 0    50   Input ~ 0
 IN_USER2
-NoConn ~ 4950 3050
 Text GLabel 4850 3150 0    50   Input ~ 0
 IN_DIFFPRES
@@
 F 0 "AIRTEC1" V 9322 6080 50  0000 L CNN
 F 1 "AIRTEC" V 9413 6080 50  0000 L CNN
-F 2 "WaveGlide3X:Airtec_M20" H 9450 6000 50  0001 C CNN
+F 2 "WaveGlide3X:Airtec_M20_B" H 9450 6000 50  0001 C CNN
 F 3 "~" H 9450 6000 50  0001 C CNN
 	1    9450 6000
@@
 Wire Wire Line
 	6500 4500 6650 4500
+$Comp
+L Connector_Generic:Conn_02x02_Counter_Clockwise VALVESSR2
+U 1 1 5E210121
+P 10300 3550
+F 0 "VALVESSR2" H 10350 3750 50  0000 C CNN
+F 1 "VALVESSR" H 10350 3676 50  0001 C CNN
+F 2 "WaveGlide3X:SSR" H 10300 3550 50  0001 C CNN
+F 3 "~" H 10300 3550 50  0001 C CNN
+	1    10300 3550
+	0    1    1    0
+$EndComp
+Wire Wire Line
+	9350 3950 10300 3950
+Wire Wire Line
+	10300 3950 10300 3850
+Wire Wire Line
+	10200 3850 9650 3850
+Wire Wire Line
+	9650 3850 9650 3800
+$Comp
+L Device:R R8
+U 1 1 5E21FDA7
+P 10300 3100
+F 0 "R8" V 10200 3100 50  0000 C CNN
+F 1 "360" V 10300 3100 50  0000 C CNN
+F 2 "Resistors_ThroughHole:R_Axial_DIN0207_L6.3mm_D2.5mm_P10.16mm_Horizontal" V 10230 3100 50  0001 C CNN
+F 3 "~" H 10300 3100 50  0001 C CNN
+	1    10300 3100
+	-1   0    0    1
+$EndComp
+Wire Wire Line
+	10200 3350 8900 3350
+Wire Wire Line
+	8900 3350 8900 3800
+Connection ~ 8900 3800
+Wire Wire Line
+	10300 3250 10300 3350
+Text GLabel 10300 2850 1    50   Input ~ 0
+OUT_VCONV
+Wire Wire Line
+	10300 2850 10300 2950
+Text GLabel 4850 3050 0    50   Output ~ 0
+OUT_VCONV
+Wire Wire Line
+	4950 3050 4850 3050
 $EndSCHEMATC

Commit message: as finished for 3X v3.1
Parts:
- AIRTEC1: footprint WaveGlide3X:Airtec_M20_B -> WaveGlide3X:Airtec_M20_B_1MH
Changed lines of the file:
@@
 F 0 "AIRTEC1" V 9322 6080 50  0000 L CNN
 F 1 "AIRTEC" V 9413 6080 50  0000 L CNN
-F 2 "WaveGlide3X:Airtec_M20_B" H 9450 6000 50  0001 C CNN
+F 2 "WaveGlide3X:Airtec_M20_B_1MH" H 9450 6000 50  0001 C CNN
 F 3 "~" H 9450 6000 50  0001 C CNN
 	1    9450 6000
